Commit message: Added comm_layer and fixed some stability issues

File: ros2_ws/src/ugv_description/urdf/ugv.urdf.xacro (robot description, xacro)
@@ -65,69 +65,3 @@
     <axis xyz="0 1 0"/>
   </joint>
-</robot><?xml version="1.0"?>
-<robot name="ugv" xmlns:xacro="http://www.ros.org/wiki/xacro">
-  <!-- Root -->
-  <link name="world"/>
-  <!-- Base -->
-  <link name="base_link">
-    <inertial>
-      <origin xyz="0 0 0" rpy="0 0 0"/>
-      <mass value="8.0"/>
-      <inertia ixx="0.25" ixy="0" ixz="0" iyy="0.35" iyz="0" izz="0.45"/>
-    </inertial>
-    <visual>
-      <geometry>
-        <box size="0.5 0.35 0.18"/>
-      </geometry>
-      <material name="blue">
-        <color rgba="0.2 0.3 0.8 1.0"/>
-      </material>
-    </visual>
-    <collision>
-      <geometry>
-        <box size="0.5 0.35 0.18"/>
-      </geometry>
-    </collision>
-  </link>
-  <!-- world -> base_link -->
-  <joint name="world_to_base" type="fixed">
-    <parent link="world"/>
-    <child link="base_link"/>
-    <origin xyz="0 0 0" rpy="0 0 0"/>
-  </joint>
-  <!-- Wheels (visual only in RViz; Gazebo will use SDF diff drive) -->
-  <link name="left_wheel_link">
-    <visual>
-      <origin xyz="0 0 0" rpy="1.5708 0 0"/>
-      <geometry>
-        <cylinder radius="0.08" length="0.04"/>
-      </geometry>
-      <material name="black">
-        <color rgba="0.1 0.1 0.1 1.0"/>
-      </material>
-    </visual>
-  </link>
-  <link name="right_wheel_link">
-    <visual>
-      <origin xyz="0 0 0" rpy="1.5708 0 0"/>
-      <geometry>
-        <cylinder radius="0.08" length="0.04"/>
-      </geometry>
-      <material name="black">
-        <color rgba="0.1 0.1 0.1 1.0"/>
-      </material>
-    </visual>
-  </link>
-  <joint name="left_wheel_joint" type="continuous">
-    <parent link="base_link"/>
-    <child link="left_wheel_link"/>
-    <origin xyz="0.0 0.19 -0.08" rpy="0 0 0"/>
-    <axis xyz="0 1 0"/>
-  </joint>
-  <joint name="right_wheel_joint" type="continuous">
-    <parent link="base_link"/>
-    <child link="right_wheel_link"/>
-    <origin xyz="0.0 -0.19 -0.08" rpy="0 0 0"/>
-    <axis xyz="0 1 0"/>
-  </joint>
 </robot>
