Commit message: Fix UAV visibility and improve world visuals for Phase 1 baseline
- Fix UAV URDF: remove world root link that prevented proper Gazebo spawning
- Embed UAV as static model in world SDF to avoid SceneBroadcaster race condition
- Add uav.sdf to uav_description/models for future dynamic spawning
- Position UAV at (-2, 0, 5) directly above UGV spawn point
- Add colors to all world elements: asphalt ground, concrete barriers,
  terracotta obstacle blocks, silver UAV, green UGV body, dark rubber wheels
- Add .gitignore for ROS 2 build artifacts, Python cache, and IDE files

Co-Authored-By: Claude Sonnet 4.6 <noreply@anthropic.com>

File: ros2_ws/src/uav_description/urdf/uav.urdf.xacro (robot description, xacro)
@@ -1,6 +1,4 @@
 <?xml version="1.0"?>
 <robot name="uav" xmlns:xacro="http://www.ros.org/wiki/xacro">
-  <!-- Root frame-->
-  <link name="world"/>
   <!-- UAV body -->
   <link name="base_link">
@@ -26,9 +24,3 @@
     </collision>
   </link>
-  <!-- Publish a transform world -> base_link -->
-  <joint name="world_to_base" type="fixed">
-    <parent link="world"/>
-    <child link="base_link"/>
-    <origin xyz="0 0 0" rpy="0 0 0"/>
-  </joint>
 </robot>

Commit message: feat: realistic MRTA scenario with APF obstacle avoidance
- Cluster UGVs at south-center (0,-7), (1,-7), (-1,-7) — realistic
  co-deployment; replaces spread start positions
- Reposition targets behind obstacle columns
- Add APF obstacle avoidance to ugv_goal_follower_node: AABB repulsion
  from hardcoded SDF geometry, robot radius inflation, turn-then-drive
  heading from resultant force vector
- Replace timer-based target observer with logical-camera-driven publish;
  add logical_camera_bridge to launch for Gazebo→ROS topic
- Add UAV quadcopter visual + logical camera sensor to uav.sdf/xacro

Co-Authored-By: Claude Sonnet 4.6 <noreply@anthropic.com>

File: ros2_ws/src/uav_description/urdf/uav.urdf.xacro (robot description, xacro)
@@ -1,5 +1,4 @@
 <?xml version="1.0"?>
 <robot name="uav" xmlns:xacro="http://www.ros.org/wiki/xacro">
-  <!-- UAV body -->
   <link name="base_link">
     <inertial>
@@ -8,18 +7,55 @@
       <inertia ixx="0.02" ixy="0.0" ixz="0.0" iyy="0.02" iyz="0.0" izz="0.04"/>
     </inertial>
+    <!-- Central body -->
     <visual>
       <origin xyz="0 0 0" rpy="0 0 0"/>
-      <geometry>
-        <box size="0.4 0.4 0.1"/>
-      </geometry>
-      <material name="gray">
-        <color rgba="0.6 0.6 0.6 1.0"/>
+      <geometry><cylinder radius="0.12" length="0.04"/></geometry>
+      <material name="body_dark">
+        <color rgba="0.30 0.30 0.33 1.0"/>
       </material>
+    </visual>
+    <!-- Arm NE-SW -->
+    <visual>
+      <origin xyz="0 0 0" rpy="0 0 0.7854"/>
+      <geometry><box size="0.56 0.03 0.015"/></geometry>
+      <material name="arm_dark">
+        <color rgba="0.27 0.27 0.30 1.0"/>
+      </material>
+    </visual>
+    <!-- Arm NW-SE -->
+    <visual>
+      <origin xyz="0 0 0" rpy="0 0 -0.7854"/>
+      <geometry><box size="0.56 0.03 0.015"/></geometry>
+      <material name="arm_dark"/>
+    </visual>
+    <!-- Rotor NE -->
+    <visual>
+      <origin xyz="0.198 0.198 0.012" rpy="0 0 0"/>
+      <geometry><cylinder radius="0.10" length="0.008"/></geometry>
+      <material name="rotor_gray">
+        <color rgba="0.60 0.60 0.65 1.0"/>
+      </material>
+    </visual>
+    <!-- Rotor NW -->
+    <visual>
+      <origin xyz="-0.198 0.198 0.012" rpy="0 0 0"/>
+      <geometry><cylinder radius="0.10" length="0.008"/></geometry>
+      <material name="rotor_gray"/>
+    </visual>
+    <!-- Rotor SW -->
+    <visual>
+      <origin xyz="-0.198 -0.198 0.012" rpy="0 0 0"/>
+      <geometry><cylinder radius="0.10" length="0.008"/></geometry>
+      <material name="rotor_gray"/>
+    </visual>
+    <!-- Rotor SE -->
+    <visual>
+      <origin xyz="0.198 -0.198 0.012" rpy="0 0 0"/>
+      <geometry><cylinder radius="0.10" length="0.008"/></geometry>
+      <material name="rotor_gray"/>
     </visual>
     <collision>
       <origin xyz="0 0 0" rpy="0 0 0"/>
-      <geometry>
-        <box size="0.4 0.4 0.1"/>
-      </geometry>
+      <geometry><cylinder radius="0.12" length="0.04"/></geometry>
     </collision>
   </link>
